Commit message: unfinished gazebo teleop

File: src/main_pkg/description/robot.urdf.xacro (robot description, xacro)
@@ -2,3 +2,4 @@
 <robot name="mars_rover" xmlns:xacro="http://www.ros.org/wiki/xacro">
     <xacro:include filename="robot_core.xacro"/>
+    <xacro:include filename="gazebo_control.xacro"/>
 </robot>

File: src/main_pkg/description/robot_core.xacro (robot description, xacro)
@@ -41,4 +41,7 @@
         </xacro:inertial_box>
     </link>
+    <gazebo reference="chassis">
+        <material>Gazebo/White</material>
+    </gazebo>
     <!-- FRONT LEFT WHEEL LINK -->
     <joint name="front_left_wheel_joint" type="continuous">
@@ -66,4 +69,7 @@
         </xacro:inertial_cylinder>
     </link>
+    <gazebo reference="front_left_wheel">
+        <material>Gazebo/Blue</material>
+    </gazebo>
         <!-- FRONT RIGHT WHEEL LINK -->
     <joint name="front_right_wheel_joint" type="continuous">
@@ -91,4 +97,7 @@
         </xacro:inertial_cylinder>
     </link>
+    <gazebo reference="front_right_wheel">
+        <material>Gazebo/Blue</material>
+    </gazebo>
         <!-- BACK LEFT WHEEL LINK -->
     <joint name="back_left_wheel_joint" type="continuous">
@@ -116,4 +125,7 @@
         </xacro:inertial_cylinder>
     </link>
+    <gazebo reference="back_left_wheel">
+        <material>Gazebo/Blue</material>
+    </gazebo>
         <!-- BACK RIGHT WHEEL LINK -->
     <joint name="back_right_wheel_joint" type="continuous">
@@ -141,3 +153,6 @@
         </xacro:inertial_cylinder>
     </link>
+    <gazebo reference="back_right_wheel">
+        <material>Gazebo/Blue</material>
+    </gazebo>
 </robot>
