Commit message: fixed lidar on robot description

File: src/main_pkg/description/gazebo_control.xacro (robot description, xacro)
@@ -2,5 +2,5 @@
 <robot name="mars_rover" xmlns:xacro="http://www.ros.org/wiki/xacro">
     <gazebo>
-        <plugin name="skid_steer_drive" filename="libgazebo_ros_diff_drive.so">
+        <plugin name="diff_drive" filename="libgazebo_ros_diff_drive.so">
             <!-- Wheel Information -->
             <num_wheel_pairs>2</num_wheel_pairs>

File: src/main_pkg/description/lidar.xacro (robot description, xacro)
@@ -1,8 +1,34 @@
 <?xml version="1.0"?>
 <robot name="mars_rover" xmlns:xacro="http://www.ros.org/wiki/xacro">
+    <joint name="laser_base_joint" type="fixed">
+        <parent link="chassis"/>
+        <child link="laser_base"/>
+        <origin xyz="0.05 0.05 0.0675" rpy="0 0 0"/>
+    </joint>
+    <link name="laser_base">
+        <visual>
+            <origin xyz="0 0 0" rpy="0 0 0"/>
+            <geometry>
+                <cylinder radius="0.015" length="0.055"/>
+            </geometry>
+            <material name="orange"/>
+        </visual>
+        <collision>
+            <origin xyz="0 0 0" rpy="0 0 0"/>
+            <geometry>
+                <cylinder radius="0.015" length="0.055"/>
+            </geometry>
+        </collision>
+        <xacro:inertial_cylinder mass="0.2" length="0.055" radius="0.015">
+            <origin xyz="0 0 0" rpy="0 0 0"/>
+        </xacro:inertial_cylinder>
+    </link>
+    <Gazebo reference="laser_base">
+        <material>Gazebo/Orange</material>
+    </Gazebo>
     <joint name="laser_joint" type="fixed">
-        <parent link="chassis"/>
+        <parent link="laser_base"/>
         <child link="laser_frame"/>
-        <origin xyz="0.1 0.1 0.2" rpy="0 0 0"/>
+        <origin xyz="0 0 0.0425" rpy="0 0 0"/>
     </joint>
     <link name="laser_frame">
@@ -10,5 +36,5 @@
             <origin xyz="0 0 0" rpy="0 0 0"/>
             <geometry>
-                <cylinder radius="0.060325" length="0.034925"/>
+                <cylinder radius="0.035" length="0.03"/>
             </geometry>
             <material name="red"/>
@@ -17,8 +43,8 @@
             <origin xyz="0 0 0" rpy="0 0 0"/>
             <geometry>
-                <cylinder radius="0.060325" length="0.034925"/>
+                <cylinder radius="0.035" length="0.03"/>
             </geometry>
         </collision>
-        <xacro:inertial_cylinder mass="0.2" length="0.034925" radius="0.060325">
+        <xacro:inertial_cylinder mass="0.2" length="0.035" radius="0.03">
             <origin xyz="0 0 0" rpy="0 0 0"/>
         </xacro:inertial_cylinder>

File: src/main_pkg/description/robot_core.xacro (robot description, xacro)
@@ -30,5 +30,5 @@
             <origin xyz="0 0 0"/>
             <geometry>
-                <box size="0.24765 0.2032 0.1016"/>
+                <box size="0.24765 0.2032 0.08"/>
             </geometry>
             <material name="white"/>
@@ -37,8 +37,8 @@
             <origin xyz="0 0 0"/>
             <geometry>
-                <box size="0.24765 0.2032 0.1016"/>
+                <box size="0.24765 0.2032 0.08"/>
             </geometry>
         </collision>
-        <xacro:inertial_box mass="0.7" x="0.24765" y="0.2032" z="0.1016">
+        <xacro:inertial_box mass="0.7" x="0.24765" y="0.2032" z="0.08">
             <origin xyz="0 0 0" rpy="0 0 0"/>
         </xacro:inertial_box>

Commit message: urdf tweaks

File: src/main_pkg/description/gazebo_control.xacro (robot description, xacro)
@@ -12,8 +12,8 @@
             <right_joint>back_right_wheel_joint</right_joint>
             <!-- One value per pair -->
-            <wheel_separation>0.238125</wheel_separation>
-            <wheel_separation>0.238125</wheel_separation>
-            <wheel_diameter>0.12065</wheel_diameter>
-            <wheel_diameter>0.12065</wheel_diameter>
+            <wheel_separation>0.2775</wheel_separation>
+            <wheel_separation>0.2775</wheel_separation>
+            <wheel_diameter>0.125</wheel_diameter>
+            <wheel_diameter>0.125</wheel_diameter>
             <!-- Limits -->
              <max_wheel_torque>200</max_wheel_torque>

File: src/main_pkg/description/robot_core.xacro (robot description, xacro)
@@ -32,5 +32,5 @@
         <parent link="base_link"/>
         <child link="chassis"/>
-        <origin xyz="0 0 0.060325"/>
+        <origin xyz="0 0 0.0625"/>
     </joint>
     <link name="chassis">
@@ -59,5 +59,5 @@
         <parent link="chassis"/>
         <child link="front_left_wheel"/>
-        <origin xyz="0.092075 0.1190625 0" rpy="0 0 0"/>
+        <origin xyz="0.092075 0.13875 0" rpy="0 0 0"/>
         <axis xyz="0 1 0"/>
     </joint>
@@ -66,5 +66,5 @@
             <origin xyz="0 0 0" rpy="1.5708 0 0"/>
             <geometry>
-                <cylinder radius="0.060325" length="0.034925"/>
+                <cylinder radius="0.0625" length="0.034925"/>
             </geometry>
             <material name="blue"/>
@@ -73,8 +73,8 @@
             <origin xyz="0 0 0" rpy="1.5708 0 0"/>
             <geometry>
-                <cylinder radius="0.060325" length="0.034925"/>
+                <cylinder radius="0.0625" length="0.034925"/>
             </geometry>
         </collision>
-        <xacro:inertial_cylinder mass="0.2" length="0.034925" radius="0.060325">
+        <xacro:inertial_cylinder mass="0.2" length="0.034925" radius="0.0625">
             <origin xyz="0 0 0" rpy="1.5708 0 0"/>
         </xacro:inertial_cylinder>
@@ -87,5 +87,5 @@
         <parent link="chassis"/>
         <child link="front_right_wheel"/>
-        <origin xyz="0.092075 -0.1190625 0" rpy="0 0 0"/>
+        <origin xyz="0.092075 -0.13875 0" rpy="0 0 0"/>
         <axis xyz="0 1 0"/>
     </joint>
@@ -94,5 +94,5 @@
             <origin xyz="0 0 0" rpy="1.5708 0 0"/>
             <geometry>
-                <cylinder radius="0.060325" length="0.034925"/>
+                <cylinder radius="0.0625" length="0.034925"/>
             </geometry>
             <material name="blue"/>
@@ -101,8 +101,8 @@
             <origin xyz="0 0 0" rpy="1.5708 0 0"/>
             <geometry>
-                <cylinder radius="0.060325" length="0.034925"/>
+                <cylinder radius="0.0625" length="0.034925"/>
             </geometry>
         </collision>
-        <xacro:inertial_cylinder mass="0.2" length="0.034925" radius="0.060325">
+        <xacro:inertial_cylinder mass="0.2" length="0.034925" radius="0.0625">
             <origin xyz="0 0 0" rpy="1.5708 0 0"/>
         </xacro:inertial_cylinder>
@@ -115,5 +115,5 @@
         <parent link="chassis"/>
         <child link="back_left_wheel"/>
-        <origin xyz="-0.092075 0.1190625 0" rpy="0 0 0"/>
+        <origin xyz="-0.092075 0.13875 0" rpy="0 0 0"/>
         <axis xyz="0 1 0"/>
     </joint>
@@ -122,5 +122,5 @@
             <origin xyz="0 0 0" rpy="1.5708 0 0"/>
             <geometry>
-                <cylinder radius="0.060325" length="0.034925"/>
+                <cylinder radius="0.0625" length="0.034925"/>
             </geometry>
             <material name="blue"/>
@@ -129,8 +129,8 @@
             <origin xyz="0 0 0" rpy="1.5708 0 0"/>
             <geometry>
-                <cylinder radius="0.060325" length="0.034925"/>
+                <cylinder radius="0.0625" length="0.034925"/>
             </geometry>
         </collision>
-        <xacro:inertial_cylinder mass="0.2" length="0.034925" radius="0.060325">
+        <xacro:inertial_cylinder mass="0.2" length="0.034925" radius="0.0625">
             <origin xyz="0 0 0" rpy="1.5708 0 0"/>
         </xacro:inertial_cylinder>
@@ -143,5 +143,5 @@
         <parent link="chassis"/>
         <child link="back_right_wheel"/>
-        <origin xyz="-0.092075 -0.1190625 0" rpy="0 0 0"/>
+        <origin xyz="-0.092075 -0.13875 0" rpy="0 0 0"/>
         <axis xyz="0 1 0"/>
     </joint>
@@ -150,5 +150,5 @@
             <origin xyz="0 0 0" rpy="1.5708 0 0"/>
             <geometry>
-                <cylinder radius="0.060325" length="0.034925"/>
+                <cylinder radius="0.0625" length="0.034925"/>
             </geometry>
             <material name="blue"/>
@@ -157,8 +157,8 @@
             <origin xyz="0 0 0" rpy="1.5708 0 0"/>
             <geometry>
-                <cylinder radius="0.060325" length="0.034925"/>
+                <cylinder radius="0.0625" length="0.034925"/>
             </geometry>
         </collision>
-        <xacro:inertial_cylinder mass="0.2" length="0.034925" radius="0.060325">
+        <xacro:inertial_cylinder mass="0.2" length="0.034925" radius="0.0625">
             <origin xyz="0 0 0" rpy="1.5708 0 0"/>
         </xacro:inertial_cylinder>

Commit message: urdf tweaks again

File: src/main_pkg/description/gazebo_control.xacro (robot description, xacro)
@@ -12,8 +12,8 @@
             <right_joint>back_right_wheel_joint</right_joint>
             <!-- One value per pair -->
-            <wheel_separation>0.2775</wheel_separation>
-            <wheel_separation>0.2775</wheel_separation>
-            <wheel_diameter>0.125</wheel_diameter>
-            <wheel_diameter>0.125</wheel_diameter>
+            <wheel_separation>0.2428</wheel_separation>
+            <wheel_separation>0.2428</wheel_separation>
+            <wheel_diameter>0.1182</wheel_diameter>
+            <wheel_diameter>0.1182</wheel_diameter>
             <!-- Limits -->
              <max_wheel_torque>200</max_wheel_torque>

File: src/main_pkg/description/robot_core.xacro (robot description, xacro)
@@ -32,5 +32,5 @@
         <parent link="base_link"/>
         <child link="chassis"/>
-        <origin xyz="0 0 0.0625"/>
+        <origin xyz="0 0 0.0591"/>
     </joint>
     <link name="chassis">
@@ -59,5 +59,5 @@
         <parent link="chassis"/>
         <child link="front_left_wheel"/>
-        <origin xyz="0.092075 0.13875 0" rpy="0 0 0"/>
+        <origin xyz="0.092075 0.1214 0" rpy="0 0 0"/>
         <axis xyz="0 1 0"/>
     </joint>
@@ -66,5 +66,5 @@
             <origin xyz="0 0 0" rpy="1.5708 0 0"/>
             <geometry>
-                <cylinder radius="0.0625" length="0.034925"/>
+                <cylinder radius="0.0591" length="0.034925"/>
             </geometry>
             <material name="blue"/>
@@ -73,8 +73,8 @@
             <origin xyz="0 0 0" rpy="1.5708 0 0"/>
             <geometry>
-                <cylinder radius="0.0625" length="0.034925"/>
+                <cylinder radius="0.0591" length="0.034925"/>
             </geometry>
         </collision>
-        <xacro:inertial_cylinder mass="0.2" length="0.034925" radius="0.0625">
+        <xacro:inertial_cylinder mass="0.2" length="0.034925" radius="0.0591">
             <origin xyz="0 0 0" rpy="1.5708 0 0"/>
         </xacro:inertial_cylinder>
@@ -87,5 +87,5 @@
         <parent link="chassis"/>
         <child link="front_right_wheel"/>
-        <origin xyz="0.092075 -0.13875 0" rpy="0 0 0"/>
+        <origin xyz="0.092075 -0.1214 0" rpy="0 0 0"/>
         <axis xyz="0 1 0"/>
     </joint>
@@ -94,5 +94,5 @@
             <origin xyz="0 0 0" rpy="1.5708 0 0"/>
             <geometry>
-                <cylinder radius="0.0625" length="0.034925"/>
+                <cylinder radius="0.0591" length="0.034925"/>
             </geometry>
             <material name="blue"/>
@@ -101,8 +101,8 @@
             <origin xyz="0 0 0" rpy="1.5708 0 0"/>
             <geometry>
-                <cylinder radius="0.0625" length="0.034925"/>
+                <cylinder radius="0.0591" length="0.034925"/>
             </geometry>
         </collision>
-        <xacro:inertial_cylinder mass="0.2" length="0.034925" radius="0.0625">
+        <xacro:inertial_cylinder mass="0.2" length="0.034925" radius="0.0591">
             <origin xyz="0 0 0" rpy="1.5708 0 0"/>
         </xacro:inertial_cylinder>
@@ -115,5 +115,5 @@
         <parent link="chassis"/>
         <child link="back_left_wheel"/>
-        <origin xyz="-0.092075 0.13875 0" rpy="0 0 0"/>
+        <origin xyz="-0.092075 0.1214 0" rpy="0 0 0"/>
         <axis xyz="0 1 0"/>
     </joint>
@@ -122,5 +122,5 @@
             <origin xyz="0 0 0" rpy="1.5708 0 0"/>
             <geometry>
-                <cylinder radius="0.0625" length="0.034925"/>
+                <cylinder radius="0.0591" length="0.034925"/>
             </geometry>
             <material name="blue"/>
@@ -129,8 +129,8 @@
             <origin xyz="0 0 0" rpy="1.5708 0 0"/>
             <geometry>
-                <cylinder radius="0.0625" length="0.034925"/>
+                <cylinder radius="0.0591" length="0.034925"/>
             </geometry>
         </collision>
-        <xacro:inertial_cylinder mass="0.2" length="0.034925" radius="0.0625">
+        <xacro:inertial_cylinder mass="0.2" length="0.034925" radius="0.0591">
             <origin xyz="0 0 0" rpy="1.5708 0 0"/>
         </xacro:inertial_cylinder>
@@ -143,5 +143,5 @@
         <parent link="chassis"/>
         <child link="back_right_wheel"/>
-        <origin xyz="-0.092075 -0.13875 0" rpy="0 0 0"/>
+        <origin xyz="-0.092075 -0.1214 0" rpy="0 0 0"/>
         <axis xyz="0 1 0"/>
     </joint>
@@ -150,5 +150,5 @@
             <origin xyz="0 0 0" rpy="1.5708 0 0"/>
             <geometry>
-                <cylinder radius="0.0625" length="0.034925"/>
+                <cylinder radius="0.0591" length="0.034925"/>
             </geometry>
             <material name="blue"/>
@@ -157,8 +157,8 @@
             <origin xyz="0 0 0" rpy="1.5708 0 0"/>
             <geometry>
-                <cylinder radius="0.0625" length="0.034925"/>
+                <cylinder radius="0.0591" length="0.034925"/>
             </geometry>
         </collision>
-        <xacro:inertial_cylinder mass="0.2" length="0.034925" radius="0.0625">
+        <xacro:inertial_cylinder mass="0.2" length="0.034925" radius="0.0591">
             <origin xyz="0 0 0" rpy="1.5708 0 0"/>
         </xacro:inertial_cylinder>

Commit message: tweaks

File: src/main_pkg/description/gazebo_control.xacro (robot description, xacro)
@@ -12,8 +12,8 @@
             <right_joint>back_right_wheel_joint</right_joint>
             <!-- One value per pair -->
-            <wheel_separation>0.2428</wheel_separation>
-            <wheel_separation>0.2428</wheel_separation>
-            <wheel_diameter>0.1182</wheel_diameter>
-            <wheel_diameter>0.1182</wheel_diameter>
+            <wheel_separation>0.238125</wheel_separation>
+            <wheel_separation>0.238125</wheel_separation>
+            <wheel_diameter>0.12065</wheel_diameter>
+            <wheel_diameter>0.12065</wheel_diameter>
             <!-- Limits -->
              <max_wheel_torque>200</max_wheel_torque>

File: src/main_pkg/description/robot_core.xacro (robot description, xacro)
@@ -32,5 +32,5 @@
         <parent link="base_link"/>
         <child link="chassis"/>
-        <origin xyz="0 0 0.0591"/>
+        <origin xyz="0 0 0.060325"/>
     </joint>
     <link name="chassis">
@@ -59,5 +59,5 @@
         <parent link="chassis"/>
         <child link="front_left_wheel"/>
-        <origin xyz="0.092075 0.1214 0" rpy="0 0 0"/>
+        <origin xyz="0.092075 0.1190625 0" rpy="0 0 0"/>
         <axis xyz="0 1 0"/>
     </joint>
@@ -66,5 +66,5 @@
             <origin xyz="0 0 0" rpy="1.5708 0 0"/>
             <geometry>
-                <cylinder radius="0.0591" length="0.034925"/>
+                <cylinder radius="0.060325" length="0.034925"/>
             </geometry>
             <material name="blue"/>
@@ -73,8 +73,8 @@
             <origin xyz="0 0 0" rpy="1.5708 0 0"/>
             <geometry>
-                <cylinder radius="0.0591" length="0.034925"/>
+                <cylinder radius="0.060325" length="0.034925"/>
             </geometry>
         </collision>
-        <xacro:inertial_cylinder mass="0.2" length="0.034925" radius="0.0591">
+        <xacro:inertial_cylinder mass="0.2" length="0.034925" radius="0.060325">
             <origin xyz="0 0 0" rpy="1.5708 0 0"/>
         </xacro:inertial_cylinder>
@@ -87,5 +87,5 @@
         <parent link="chassis"/>
         <child link="front_right_wheel"/>
-        <origin xyz="0.092075 -0.1214 0" rpy="0 0 0"/>
+        <origin xyz="0.092075 -0.1190625 0" rpy="0 0 0"/>
         <axis xyz="0 1 0"/>
     </joint>
@@ -94,5 +94,5 @@
             <origin xyz="0 0 0" rpy="1.5708 0 0"/>
             <geometry>
-                <cylinder radius="0.0591" length="0.034925"/>
+                <cylinder radius="0.060325" length="0.034925"/>
             </geometry>
             <material name="blue"/>
@@ -101,8 +101,8 @@
             <origin xyz="0 0 0" rpy="1.5708 0 0"/>
             <geometry>
-                <cylinder radius="0.0591" length="0.034925"/>
+                <cylinder radius="0.060325" length="0.034925"/>
             </geometry>
         </collision>
-        <xacro:inertial_cylinder mass="0.2" length="0.034925" radius="0.0591">
+        <xacro:inertial_cylinder mass="0.2" length="0.034925" radius="0.060325">
             <origin xyz="0 0 0" rpy="1.5708 0 0"/>
         </xacro:inertial_cylinder>
@@ -115,5 +115,5 @@
         <parent link="chassis"/>
         <child link="back_left_wheel"/>
-        <origin xyz="-0.092075 0.1214 0" rpy="0 0 0"/>
+        <origin xyz="-0.092075 0.1190625 0" rpy="0 0 0"/>
         <axis xyz="0 1 0"/>
     </joint>
@@ -122,5 +122,5 @@
             <origin xyz="0 0 0" rpy="1.5708 0 0"/>
             <geometry>
-                <cylinder radius="0.0591" length="0.034925"/>
+                <cylinder radius="0.060325" length="0.034925"/>
             </geometry>
             <material name="blue"/>
@@ -129,8 +129,8 @@
             <origin xyz="0 0 0" rpy="1.5708 0 0"/>
             <geometry>
-                <cylinder radius="0.0591" length="0.034925"/>
+                <cylinder radius="0.060325" length="0.034925"/>
             </geometry>
         </collision>
-        <xacro:inertial_cylinder mass="0.2" length="0.034925" radius="0.0591">
+        <xacro:inertial_cylinder mass="0.2" length="0.034925" radius="0.060325">
             <origin xyz="0 0 0" rpy="1.5708 0 0"/>
         </xacro:inertial_cylinder>
@@ -143,5 +143,5 @@
         <parent link="chassis"/>
         <child link="back_right_wheel"/>
-        <origin xyz="-0.092075 -0.1214 0" rpy="0 0 0"/>
+        <origin xyz="-0.092075 -0.1190625 0" rpy="0 0 0"/>
         <axis xyz="0 1 0"/>
     </joint>
@@ -150,5 +150,5 @@
             <origin xyz="0 0 0" rpy="1.5708 0 0"/>
             <geometry>
-                <cylinder radius="0.0591" length="0.034925"/>
+                <cylinder radius="0.060325" length="0.034925"/>
             </geometry>
             <material name="blue"/>
@@ -157,8 +157,8 @@
             <origin xyz="0 0 0" rpy="1.5708 0 0"/>
             <geometry>
-                <cylinder radius="0.0591" length="0.034925"/>
+                <cylinder radius="0.060325" length="0.034925"/>
             </geometry>
         </collision>
-        <xacro:inertial_cylinder mass="0.2" length="0.034925" radius="0.0591">
+        <xacro:inertial_cylinder mass="0.2" length="0.034925" radius="0.060325">
             <origin xyz="0 0 0" rpy="1.5708 0 0"/>
         </xacro:inertial_cylinder>
