Commit message: lidar urdf fix

File: src/main_pkg/description/lidar.xacro (robot description, xacro)
@@ -4,5 +4,5 @@
         <parent link="chassis"/>
         <child link="laser_base"/>
-        <origin xyz="0.05 0.05 0.0675" rpy="0 0 0"/>
+        <origin xyz="0.05 0.05 0.0675" rpy="0 0 3.14159"/>
     </joint>
     <link name="laser_base">
